File: cap-touch-sensor/cap-touch-sensor.kicad_sch (KiCad schematic)
At the start: 10 parts, among them U3 TTP223-BA6

Commit message: Update CAD files and gitignore
Parts:
- removed JP2, JP3: SolderJumper_2_Bridged, Jumper:SolderJumper-2_P1.3mm_Bridged_RoundedPad1.0x1.5mm, symbol Jumper:SolderJumper_2_Bridged
- removed TP1: Vcc, TestPoint:TestPoint_Pad_1.5x1.5mm, symbol Connector:TestPoint
- removed TP2: TOGGLE, TestPoint:TestPoint_Pad_1.5x1.5mm, symbol Connector:TestPoint
- removed TP3: GND, TestPoint:TestPoint_Pad_1.5x1.5mm, symbol Connector:TestPoint
- added J1: VBAT, Connector_PinHeader_1.27mm:PinHeader_1x01_P1.27mm_Vertical, symbol Connector:Conn_01x01_Pin
- added J2: TOG, Connector_PinHeader_1.27mm:PinHeader_1x01_P1.27mm_Vertical, symbol Connector:Conn_01x01_Pin
- added J3: GND, Connector_PinHeader_1.27mm:PinHeader_1x01_P1.27mm_Vertical, symbol Connector:Conn_01x01_Pin
- added JP2: SolderJumper_2_Open, Jumper:SolderJumper-2_P1.3mm_Open_RoundedPad1.0x1.5mm, symbol Jumper:SolderJumper_2_Open
- C5, C6: footprint Capacitor_SMD:C_0805_2012Metric -> Capacitor_SMD:C_0603_1608Metric
Connections:
- net GND: now also U3.4 (AHLB), J3.1 (Pin_1), JP2.1 (A)
- net TOGGLE: now also J2.1 (Pin_1)
- net VBAT: now also J1.1 (Pin_1)
- net at U3.6 (TOG): now also JP1.1 (A), JP2.2 (B)
Other:
- moved on the sheet: JP1
