File: FancyLight-V2.kicad_pcb (KiCad board)
At the start: 2 copper layers, 40 x 40 mm, 51 parts, among them J1 PWR, Q1 IRLML2402, SW1 ONOFF, U1 SB6286, U2 TP4056, U3 TTP223-BA6, U4 DW01-P, U5 CJL8205A

Commit message: WIP
Parts:
- removed ? (x4): , 
- removed C7: 0.1u, Capacitor_SMD:C_0805_2012Metric
- removed R10: 470, Resistor_SMD:R_0805_2012Metric
- removed REF** (x2): TestPoint_THTPad_1.0x1.0mm_Drill0.5mm, TestPoint:TestPoint_THTPad_1.0x1.0mm_Drill0.5mm
- removed REF**: MountingHole_3.2mm_M3, MountingHole:MountingHole_3.2mm_M3
- removed TP1: VBAT, TestPoint:TestPoint_Pad_1.5x1.5mm
- removed TP2: GND, TestPoint:TestPoint_Pad_1.5x1.5mm
- removed TP3: TOGGLE, TestPoint:TestPoint_Pad_1.5x1.5mm
- removed TP4: SENSE, TestPoint:TestPoint_Pad_1.0x1.0mm
- removed U4: DW01-P, Package_TO_SOT_SMD:SOT-23-6
- added D10: LED, LED_SMD:LED_0603_1608Metric, F.Cu at (59.1, 65.5)
- added D7: MBR0520LT1, Diode_SMD:D_SOD-123, F.Cu at (26.6, 36.1)
- added D8: MBR0520LT1, Diode_SMD:D_SOD-123, F.Cu at (29.2, 36.2)
- added D9: RB751V-40, Diode_SMD:D_SOD-323, F.Cu at (33.2, 60.2)
- added J2: TOUCH, Connector_PinHeader_1.27mm:PinHeader_1x03_P1.27mm_Vertical, F.Cu at (20.9, 9.10)
- added J3: MODE, Connector_PinHeader_2.54mm:PinHeader_2x02_P2.54mm_Vertical, F.Cu at (11.1, 4.42)
- added Q2: IRLML2402, Package_TO_SOT_SMD:SOT-23, F.Cu at (17.5, 3.40)
- added R14: 330, Resistor_SMD:R_0603_1608Metric, F.Cu at (50.9, 58.5)
- added R15: R_Photo, Connector_PinHeader_1.27mm:PinHeader_1x02_P1.27mm_Vertical, F.Cu at (24.9, 2.50)
- added R16: 10k, Resistor_SMD:R_0603_1608Metric, B.Cu at (31.0, 4.50)
- added R17: 5k, Resistor_SMD:R_0603_1608Metric, F.Cu at (50.9, 63.6)
- added R18: 10k, Resistor_SMD:R_0603_1608Metric, F.Cu at (9.70, 9.90)
- added RN1: 330, Resistor_SMD:R_Array_Convex_4x0603, F.Cu at (25.6, 6.03)
- added U6: ATtiny44A-M, Package_DFN_QFN:QFN-20-1EP_4x4mm_P0.5mm_EP2.6x2.6mm, F.Cu at (30.4, 5.72)
- added USB1: TYPE-C_6P, kicad_lceda:TYPE-C-SMD_TYPE-C-6P, F.Cu at (20.0, 36.4)
- BT1, SW1: footprint Connector_PinHeader_2.54mm:PinHeader_2x01_P2.54mm_Vertical -> Connector_PinHeader_1.27mm:PinHeader_1x02_P1.27mm_Vertical
- C3, C4, C5: footprint Capacitor_SMD:C_0805_2012Metric -> Capacitor_SMD:C_0603_1608Metric
- C6: value 10pF (15pF) -> 0.1u; footprint Capacitor_SMD:C_0805_2012Metric -> Capacitor_SMD:C_0603_1608Metric
- D6: footprint LED_SMD:LED_1206_3216Metric -> LED_SMD:LED_0805_2012Metric
- H1, H2, H3, H4: renamed from REF**; value MountingHole_2.5mm -> ~
- J1: value PWR -> ISP; footprint Connector_USB:USB_Micro-B_Molex_47346-0001 -> Connector_PinHeader_2.54mm:PinHeader_2x03_P2.54mm_Vertical
- R11, R3, R4, R5, R6: footprint Resistor_SMD:R_0805_2012Metric -> Resistor_SMD:R_0603_1608Metric
- R12: value 100 -> 330; footprint Resistor_SMD:R_0805_2012Metric -> Resistor_SMD:R_0603_1608Metric
- R13: value 1k -> 10k; footprint Resistor_SMD:R_0805_2012Metric -> Resistor_SMD:R_0603_1608Metric
- R7: value 0 -> 5.1k; footprint Resistor_SMD:R_0805_2012Metric -> Resistor_SMD:R_0603_1608Metric
- R8, R9: value 0 -> 1k; footprint Resistor_SMD:R_0805_2012Metric -> Resistor_SMD:R_0603_1608Metric
- U3: value TTP223-BA6 -> XB3303A; footprint Package_TO_SOT_SMD:SOT-23-6 -> kicad_lceda:SOT-23-3_L2.9-W1.3-P1.90-LS2.4-BR
- U5: value CJL8205A -> syn480r; footprint Package_TO_SOT_SMD:TSOT-23-6 -> Connector_PinHeader_1.27mm:PinHeader_1x03_P1.27mm_Vertical
- moved R13 59.3 mm to (62.5, 66.1)
- moved R9 48.3 mm to (32.7, 55.9)
- moved R7 32.5 mm to (13.9, 35.2), turned to 90 degrees
- moved U3 26.3 mm to (32.1, 29.0), turned to -90 degrees
- moved J1 24.3 mm to (35.1, 18.2), turned to -90 degrees
- moved R8 23.4 mm to (34.6, 32.5)
- moved R12 22.4 mm to (21.3, 3.80), turned to 0 degrees
- moved U5 22.0 mm to (17.0, 6.53)
- moved C5 22.0 mm to (29.5, 31.5)
- moved Q1 21.6 mm to (29.5, 10.3), turned to 0 degrees
- moved C1 21.1 mm to (25.4, 19.8), turned to -90 degrees
- moved R1 19.9 mm to (-6.83, 18.3)
- moved R2 19.9 mm to (-6.81, 20.5)
- moved C6 18.3 mm to (33.1, 9.10)
- moved L1 17.3 mm to (22.8, 19.6), turned to 90 degrees
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Connections:
- net Net-(Q1-G) renamed PWM
- C3 pad 1: VCC -> Net-(D6-A)
- C5 pad 1: VBAT -> Net-(U3-VDD)
- C5 pad 2: BAT- -> Net-(BT1--)
- C6 pad 1: Net-(U3-I) -> BAT-
- C6 pad 2: BAT- -> VBAT
- D6 pad 2: VCC -> Net-(D6-A)
- J1 pad 1: VCC -> MISO
- J1 pad 2: unconnected-(J1-D--Pad2) -> VBAT
- J1 pad 3: unconnected-(J1-D+-Pad3) -> SCK
- J1 pad 4: unconnected-(J1-ID-Pad4) -> MODE1
- J1 pad 5: BAT- -> RST
- J1 pad 6: unconnected-(J1-Shield-Pad6) -> BAT-
- R12 pad 1: BAT+ -> R_EN
- R12 pad 2: Net-(U4-VCC) -> MISO
- R13 pad 1: Net-(U4-CS) -> RST
- R13 pad 2: BAT- -> VBAT
- R7 pad 1: Net-(U3-TOG) -> Net-(USB1-CC1)
- R7 pad 2: VBAT -> BAT-
- R8 pad 1: VBAT -> BAT+
- R8 pad 2: Net-(U3-AHLB) -> Net-(U3-VDD)
- R9 pad 1: Net-(U3-AHLB) -> BAT-
- R9 pad 2: BAT- -> Net-(D6-A)
- SW1 pad 1: BAT+ -> Net-(D7-K)
- U1 pad 4: TOGGLE -> DCDC_EN
- U2 pad 4: VCC -> Net-(D6-A)
- U2 pad 8: VCC -> Net-(D6-A)
- U3 pad 1: TOGGLE -> BAT-
- U3 pad 2: BAT- -> Net-(U3-VDD)
- U3 pad 3: Net-(U3-I) -> Net-(BT1--)
- U5 pad 1: BAT- -> Net-(Q2-D)
- U5 pad 2: unconnected-(U5-S1/D2-Pad2) -> R_TRIG
- U5 pad 3: Net-(BT1--) -> VBAT
Routing:
- net MODE1: track 0.00 -> 44.8 mm, vias 0 -> 1
- net TOGGLE: track 37.9 -> 0.00 mm, vias 2 -> 0
- net MISO: track 0.00 -> 31.5 mm, vias 0 -> 1
- net Net-(D6-A): track 0.00 -> 30.1 mm, vias 0 -> 2
- net VCC: track 28.0 -> 0.00 mm, vias 3 -> 0
- net SCK: track 0.00 -> 20.0 mm, vias 0 -> 1
- net DCDC_EN: track 0.00 -> 18.1 mm, vias 0 -> 2
- net VBAT: track 90.1 -> 72.9 mm, vias 2 -> 1
- net DRAIN: track 33.7 -> 16.9 mm
- net RST: track 0.00 -> 16.0 mm, vias 0 -> 1
- net Net-(U3-TOG): track 15.0 -> 0.00 mm
- net Net-(U6-PA3): track 0.00 -> 13.2 mm
- net Net-(RN1-R4.1): track 0.00 -> 12.8 mm, vias 0 -> 3
- net Net-(U3-VDD): track 0.00 -> 11.8 mm, vias 0 -> 2
- net Net-(U3-AHLB): track 11.3 -> 0.00 mm
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
Commit message: Update CAD files and gitignore
Parts:
- R16: moved to F.Cu
- moved D10 74.2 mm to (6.70, 13.1)
- moved R13 70.2 mm to (6.60, 23.6), turned to 0 degrees
- moved R17 65.1 mm to (9.80, 13.1), turned to 180 degrees
- moved R14 51.3 mm to (10.4, 27.2), turned to 0 degrees
- moved D9 37.4 mm to (11.3, 29.9), turned to -90 degrees
- moved R9 30.8 mm to (11.7, 33.4), turned to 90 degrees
- moved J1 27.8 mm to (7.30, 18.1)
- moved C6 25.5 mm to (8.20, 3.70), turned to 0 degrees
- moved J3 23.1 mm to (6.05, 26.9)
- moved R18 23.1 mm to (4.67, 32.4)
- moved R16 22.8 mm to (9.25, 11.4), turned to 180 degrees
- moved U6 21.2 mm to (9.30, 7.30), turned to 180 degrees
- moved R1 17.3 mm to (10.4, 16.9), turned to -90 degrees
- moved R2 17.2 mm to (10.2, 22.9), turned to 90 degrees
- moved RN1 11.6 mm to (14.1, 7.00), turned to 0 degrees
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Routing:
- net VBAT: track 72.9 -> 121.0 mm
- net Net-(U6-XTAL2/PB1): track 1.88 -> 32.2 mm, vias 1 -> 4
- net MODE1: track 44.8 -> 20.5 mm
- net MODE2: track 1.05 -> 24.1 mm
- net PWM: track 6.55 -> 22.5 mm, vias 0 -> 2
- net Net-(U6-PA3): track 13.2 -> 25.5 mm
- net LED_PWR: track 5.69 -> 14.4 mm
- net MISO: track 31.5 -> 23.1 mm, vias 1 -> 2
- net DCDC_EN: track 18.1 -> 24.9 mm
- net SCK: track 20.0 -> 13.9 mm, vias 1 -> 2
- net RST: track 16.0 -> 21.9 mm, vias 1 -> 0
- net Net-(U3-VDD): track 11.8 -> 6.88 mm, vias 2 -> 0
- net Net-(D6-A): track 30.1 -> 34.7 mm
- net Net-(RN1-R4.1): track 12.8 -> 8.71 mm, vias 3 -> 2
- net BAT-: track 0.00 -> 3.62 mm, vias 8 -> 24
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
Commit message: Improve schematic and PCB
Parts:
- removed L1: LQH32MN2R2K23L, lib:IND_LQH32MN2R2K23L
- removed the R14 at (10.4, 27.2)
- added C5: 10u, Capacitor_SMD:C_0603_1608Metric, F.Cu at (33.0, 6.40)
- added C7: 10u, Capacitor_SMD:C_0603_1608Metric, F.Cu at (30.8, 1.75)
- added C8: 10u, Capacitor_SMD:C_0603_1608Metric, F.Cu at (17.7, 3.20)
- added G***: LOGO, lib:logo, F.Cu at (33.9, 20.4)
- added H5: ~, MountingHole:MountingHole_2.1mm, F.Cu at (32.0, 16.0)
- added Q1: AO3400A, Package_TO_SOT_SMD:SOT-23, F.Cu at (7.96, 28.9)
- added R10: 10k, Resistor_SMD:R_0603_1608Metric, F.Cu at (4.30, 30.0)
- added R11: 10k, Resistor_SMD:R_0603_1608Metric, F.Cu at (4.30, 31.7)
- added U1: APSWPA3015S4R7MTF, kicad_lceda:IND-SMD_L3.0-W3.0, F.Cu at (23.1, 18.8)
- added U5: HT7530S_C5451677, kicad_lceda:SOT-23-3_L2.9-W1.3-P1.90-LS2.4-BR-CW, F.Cu at (30.8, 4.75)
- D10: value LED -> STATUS LED
- D5: value MBR0520LT1 (B5819W SL) -> B5819W SL
- D6: renamed from D9; value RB751V-40 -> 1N5819WS
- D7: renamed from D6; value LED -> CHRG LED; footprint LED_SMD:LED_0805_2012Metric -> LED_SMD:LED_0603_1608Metric
- D8: renamed from D7; value MBR0520LT1 -> B5819W SL
- D9: renamed from D8; value MBR0520LT1 -> B5819W SL
- Q2: renamed from Q1; value IRLML2402 -> AO3400A
- Q3: renamed from Q2; value IRLML2402 -> AO3400A
- R2: renamed from R1; value 47 -> 22
- R3: renamed from R2; value 47 -> 22
- RN1: value 330 -> 470
- moved R14 14.0 mm to (5.20, 9.70), turned to -90 degrees
- moved D10 6.58 mm to (13.1, 11.5), turned to 180 degrees
- moved J1 6.51 mm to (2.96, 13.3), turned to 0 degrees
- moved R17 5.37 mm to (13.8, 8.60), turned to 90 degrees
- moved R18 4.42 mm to (4.30, 28.0)
- moved J3 4.30 mm to (5.50, 22.7)
- moved RN1 3.48 mm to (17.6, 6.98)
- moved J2 3.48 mm to (20.9, 3.46)
- moved Q3 3.48 mm to (23.3, 9.43)
- moved R15 3.48 mm to (20.3, 9.33)
- moved R16 3.48 mm to (27.6, 3.48)
- moved U7 3.48 mm to (24.2, 6.00)
- moved Q2 3.24 mm to (30.0, 9.15), turned to 0 degrees
- moved R9 2.05 mm to (27.1, 9.05), turned to -90 degrees
- moved R13 1.19 mm to (10.7, 12.3), turned to 90 degrees
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- renumbered C3 to C1, C1 to C2, C4 to C3, C2 to C4, C5 to C6, C6 to C9, D3 to D2, D2 to D3, R5 to R1, R8 to R12, R17 to R13, R13 to R14, R12 to R15, R15 to R16, R16 to R17, R7 to R4, R9 to R5, R4 to R7, R3 to R8, R11 to R9, U1 to U2, U2 to U3, U3 to U4, U5 to U7
Connections:
- D6 pad 1: SENSE -> Net-(D6-K)
- J2 pad 1: VBAT -> 3V
- R16 pad 1: VBAT -> 3V
- R17 pad 2: SINK -> Net-(U6-PA2)
- RN1 pad 5: R_TRIG -> PWM
- RN1 pad 6: PWM -> R_TRIG
- U6 pad 12: Net-(U6-XTAL2/PB1) -> SENSE
- U6 pad 14: SINK -> Net-(RN1-R4.1)
- U6 pad 15: Net-(RN1-R4.1) -> Net-(RN1-R3.1)
- U6 pad 3: Net-(RN1-R3.1) -> Net-(U6-PA2)
Routing:
- net VBAT: track 121.0 -> 15.5 mm, vias 1 -> 7
- net Net-(U6-XTAL2/PB1): track 32.2 -> 0.00 mm, vias 4 -> 0
- net SENSE: track 1.68 -> 30.6 mm
- net 3V: track 0.00 -> 15.2 mm
- net Net-(RN1-R3.1): track 2.02 -> 15.6 mm, vias 0 -> 2
- net DCDC_EN: track 24.9 -> 38.1 mm
- net PWM: track 22.5 -> 12.3 mm
- net Net-(D6-A): track 34.7 -> 43.4 mm
- net SINK: track 7.28 -> 0.00 mm
- net RST: track 21.9 -> 15.6 mm, vias 0 -> 1
- net Net-(U6-PA3): track 25.5 -> 19.3 mm, vias 0 -> 1
- net DRAIN: track 13.5 -> 19.0 mm
- net Net-(RN1-R4.1): track 8.71 -> 14.1 mm
- net MODE1: track 20.5 -> 15.6 mm, vias 1 -> 0
- net SCK: track 13.9 -> 17.7 mm
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- added copper zone on In1.Cu, net BAT-
- added copper zone on F.Cu, net VBAT
- added copper zone on In2.Cu, net VBAT
Other:
- copper layers 2 -> 4
- board text added: "v3.1"
